File: HW/robotControlBoard.sch (KiCad schematic (older format))
At the start: 32 parts, among them P1 CONN_02X10, P2 CONN_01X03, SW1 SW_PUSH, U1 STM32F411RxT, Y1 Crystal_Small_4Pin, Y2 Crystal_Small_4Pin

Commit message: Started power design
Parts:
- added U?: LD1117S50TR, SOT-223, symbol LD1117S50TR
Connections:
- net +12V: now also U?.3 (VI)
- net GND: now also U?.1 (GND)
- new net +5V: U?.2 (VO)
Changed lines of the file:
@@
 	8200 1400 7950 1400
 Wire Wire Line
-	7400 1400 7650 1400
+	6850 1400 7650 1400
 Wire Wire Line
 	8200 1500 7950 1500
@@
 	1    0    0    -1
 $EndComp
+$Comp
+L LD1117S50TR U?
+U 1 1 596714F3
+P 6450 1450
+F 0 "U?" H 6450 1700 50  0000 C CNN
+F 1 "LD1117S50TR" H 6450 1650 50  0000 C CNN
+F 2 "SOT-223" H 6450 1550 50  0000 C CNN
+F 3 "" H 6450 1450 50  0000 C CNN
+	1    6450 1450
+	-1   0    0    -1
+$EndComp
+Connection ~ 7400 1400
+Wire Wire Line
+	6050 1400 5350 1400
+Wire Wire Line
+	5350 1400 5350 1350
+$Comp
+L GND #PWR?
+U 1 1 59671BD0
+P 6450 1700
+F 0 "#PWR?" H 6450 1450 50  0001 C CNN
+F 1 "GND" H 6450 1550 50  0000 C CNN
+F 2 "" H 6450 1700 50  0000 C CNN
+F 3 "" H 6450 1700 50  0000 C CNN
+	1    6450 1700
+	1    0    0    -1
+$EndComp
+$Comp
+L +5V #PWR?
+U 1 1 59671D8B
+P 5350 1350
+F 0 "#PWR?" H 5350 1200 50  0001 C CNN
+F 1 "+5V" H 5350 1490 50  0000 C CNN
+F 2 "" H 5350 1350 50  0000 C CNN
+F 3 "" H 5350 1350 50  0000 C CNN
+	1    5350 1350
+	1    0    0    -1
+$EndComp
